Commit message: New URDF created

File: Drone URDF/Drone/urdf/Drone.urdf (robot description, URDF)
Before this commit: robot Drone, 5 links, 4 joints
Links:
- link base_link: geometry collision mesh filename=package://drone/meshes/base_link.STL; visual mesh filename=package://drone/meshes/base_link.STL
- link wing_link1: geometry collision mesh filename=package://drone/meshes/wing_link1.STL; visual mesh filename=package://drone/meshes/wing_link1.STL
- link wing_link2: geometry collision mesh filename=package://drone/meshes/wing_link2.STL; visual mesh filename=package://drone/meshes/wing_link2.STL
- link wing_link3: geometry collision mesh filename=package://drone/meshes/wing_link3.STL; visual mesh filename=package://drone/meshes/wing_link3.STL
- link wing_link4: geometry collision mesh filename=package://drone/meshes/wing_link4.STL; visual mesh filename=package://drone/meshes/wing_link4.STL
Joints:
- removed joint joint_1
- removed joint joint_2
- removed joint joint_3
- removed joint joint_4
- added joint joint1: type revolute, parent base_link, child wing_link1, origin xyz=0.043914 -0.22904 0.12287 rpy=1.5708 0 -0.29318, axis 0 1 0, limit lower=0 upper=0 effort=0 velocity=0
- added joint joint2: type revolute, parent base_link, child wing_link2, origin xyz=-0.0033195 -0.052423 0.12287 rpy=1.5708 0 -1.6567, axis 0 1 0, limit lower=0 upper=0 effort=0 velocity=0
- added joint joint3: type revolute, parent base_link, child wing_link3, origin xyz=0.17791 -0.0047715 0.12287 rpy=1.5708 0 -3.0248, axis 0 1 0, limit lower=0 upper=0 effort=0 velocity=0
- added joint joint4: type revolute, parent base_link, child wing_link4, origin xyz=0.22366 -0.18178 0.12287 rpy=1.5708 0 0.43793, axis 0 1 0, limit lower=0 upper=0 effort=0 velocity=0
