Commit message: Added Camera and changed Joint types

File: Drone URDF/Drone/urdf/drone.urdf (robot description, URDF)
Before this commit: robot drone, 5 links, 4 joints
Links:
- added link camera_link, mass 0.00012; collision box size=0.007 0.007 0.007; visual box size=0.007 0.007 0.007
- added link camera_link_optical
Joints:
- added joint camera_joint: type fixed, parent base_link, child camera_link, origin xyz=0.10398871393486 -0.1 0.112663263182331 rpy=0 0 0, axis 0 0 1
- added joint camera_optical_joint: type fixed, parent camera_link, child camera_link_optical, origin xyz=0 0 0 rpy=-1.57079632 0 -1.57079632
- joint joint1: type revolute -> continuous
- joint joint2: type revolute -> continuous
- joint joint3: type revolute -> continuous
- joint joint4: type revolute -> continuous
