Commit message: Drone Plugin working

File: Drone URDF/drone/urdf/drone.urdf (robot description, URDF)
Before this commit: robot drone, 7 links, 6 joints
Links:
- removed link wing_link1
- removed link wing_link2
- removed link wing_link3
- removed link wing_link4
- added link prop1, mass 0.0037436; collision mesh filename=package://drone/meshes/wing_link1.STL; visual mesh filename=package://drone/meshes/wing_link1.STL
- added link prop2, mass 0.0037436; collision mesh filename=package://drone/meshes/wing_link2.STL; visual mesh filename=package://drone/meshes/wing_link2.STL
- added link prop3, mass 0.0037436; collision mesh filename=package://drone/meshes/wing_link3.STL; visual mesh filename=package://drone/meshes/wing_link3.STL
- added link prop4, mass 0.0037436; collision mesh filename=package://drone/meshes/wing_link4.STL; visual mesh filename=package://drone/meshes/wing_link4.STL
- link base_link: mass 0.126804991176584 -> 2.26804991176584
Joints:
- removed joint joint1
- removed joint joint2
- removed joint joint3
- removed joint joint4
- added joint prop1_joint: type continuous, parent base_link, child prop1, origin xyz=0.043914 -0.22904 0.12287 rpy=1.5708 0 -0.29318, axis 0 1 0, limit lower=0 upper=0 effort=0 velocity=0
- added joint prop2_joint: type continuous, parent base_link, child prop2, origin xyz=-0.0033195 -0.052423 0.12287 rpy=1.5708 0 -1.6567, axis 0 1 0, limit lower=0 upper=0 effort=0 velocity=0
- added joint prop3_joint: type continuous, parent base_link, child prop3, origin xyz=0.17791 -0.0047715 0.12287 rpy=1.5708 0 -3.0248, axis 0 1 0, limit lower=0 upper=0 effort=0 velocity=0
- added joint prop4_joint: type continuous, parent base_link, child prop4, origin xyz=0.22366 -0.18178 0.12287 rpy=1.5708 0 0.43793, axis 0 1 0, limit lower=0 upper=0 effort=0 velocity=0
